File: design/Simple008.kicad_sch (KiCad schematic)
At the start: 45 parts, among them IC1 DS1233-10+, J1 UART A, J2 UART B, J3 SD CARD, J4 Power, J5 ATF1508 JTAG, SW1 SW_Push, U1 SST39SF040, U2 AS6C8008-55ZIN, U3 MC68008, U4 XR68C681, U5 ATF1508, U6 AS6C8008-55ZIN, U7 AS6C8008-55ZIN, U8 AS6C8008-55ZIN, Y1 10MHz, Y2 3.6864MHz

Commit message: PCB layout component positioning
Parts:
- removed D2: RED, LED_SMD:LED_0805_2012Metric_Pad1.15x1.40mm_HandSolder, symbol Device:LED
- removed D3: GREEN, LED_SMD:LED_0805_2012Metric_Pad1.15x1.40mm_HandSolder, symbol Device:LED
- removed IC1: DS1233-10+, TO-92, symbol DS1233:DS1233-10+
- removed J4: Power, Connector_PinHeader_2.54mm:PinHeader_1x02_P2.54mm_Vertical, symbol Connector:Conn_01x02_Pin
- removed LED2: Halt, LED_SMD:LED_0805_2012Metric_Pad1.15x1.40mm_HandSolder, symbol rosco_m68k-eagle-import:LED5MM
- removed R1, R4: 1K, Resistor_SMD:R_0805_2012Metric_Pad1.20x1.40mm_HandSolder, symbol rosco_m68k-eagle-import:R-EU_0207_10
- removed RN3: R_Network08_Split, Resistor_THT:R_Array_SIP9, symbol Device:R_Network08_Split
- removed Run1: RED, LED_SMD:LED_0805_2012Metric_Pad1.15x1.40mm_HandSolder, symbol rosco_m68k-eagle-import:LED5MM
- removed U2, U6, U7, U8: AS6C8008-55ZIN, Package_SO:TSOP-II-44_10.16x18.41mm_P0.8mm, symbol AS6C8008-55ZIN:AS6C8008-55ZIN
- removed U3: MC68008, Package_LCC:PLCC-52_THT-Socket, symbol mackerel-68k-symbols:MC68008
- removed U4: XR68C681, Package_LCC:PLCC-44_THT-Socket, symbol mackerel-68k-symbols:XR68C681
- added H1, H2, H3, H4: MountingHole, MountingHole:MountingHole_3.2mm_M3, symbol Mechanical:MountingHole
- added IC1: DS1233-10+, Package_TO_SOT_THT:TO-92_HandSolder, symbol ds1233-10+:DS1233-10+
- added J4: Conn_02x32_Odd_Even, Connector_PinHeader_2.54mm:PinHeader_2x32_P2.54mm_Vertical, symbol Connector_Generic:Conn_02x32_Odd_Even
- added J6: Conn_01x02_Pin, Connector_PinHeader_2.54mm:PinHeader_1x02_P2.54mm_Vertical, symbol Connector:Conn_01x02_Pin
- added LED1: GREEN, LED_SMD:LED_0805_2012Metric_Pad1.15x1.40mm_HandSolder, symbol Device:LED
- added LED2: RED, LED_SMD:LED_0805_2012Metric_Pad1.15x1.40mm_HandSolder, symbol Device:LED
- added LED3: HALT, LED_SMD:LED_0805_2012Metric_Pad1.15x1.40mm_HandSolder, symbol Device:LED
- added LED4: RUN, LED_SMD:LED_0805_2012Metric_Pad1.15x1.40mm_HandSolder, symbol Device:LED
- added R1, R4: 1K, Resistor_SMD:R_0805_2012Metric_Pad1.20x1.40mm_HandSolder, symbol Device:R
- added R5: 10K, Resistor_SMD:R_0805_2012Metric_Pad1.20x1.40mm_HandSolder, symbol Device:R
- added RN1: R_Network08, Resistor_THT:R_Array_SIP9, symbol Device:R_Network08
- added U2: AS6C8008-55ZIN, Package_SO:TSOP-II-44_10.16x18.41mm_P0.8mm, symbol as6c8008:AS6C8008-55ZIN
- added U3: MC68008, Package_LCC:PLCC-52_THT-Socket, symbol mc68008:MC68008
- added U4: XR68C681, Package_LCC:PLCC-44_THT-Socket, symbol xr68c681:XR68C681
- JP1, JP2: footprint (none) -> Connector_PinHeader_2.54mm:PinHeader_1x02_P2.54mm_Vertical
- U5: symbol CPLD_Microchip:ATF1504AS-PLCC84 -> atf1508as-plcc84:ATF1508AS-PLCC84
Connections:
- net A0: now also J4.1 (Pin_1), U3.51 (A0)
- net A1: now also J4.3 (Pin_3), U2.5 (A0), U3.52 (A1), U4.2 (A1)
- net A10: now also J4.21 (Pin_21), U2.28 (A9), U3.9 (A10)
- net A11: now also J4.23 (Pin_23), U2.27 (A10), U3.10 (A11)
- net A12: now also J4.25 (Pin_25), U2.26 (A11), U3.11 (A12)
- net A13: now also J4.27 (Pin_27), U2.25 (A12), U3.12 (A13)
- net A14: now also J4.29 (Pin_29), U2.24 (A13), U3.14 (A14)
- net A15: now also J4.31 (Pin_31), U2.23 (A14), U3.16 (A15)
- net A16: now also J4.33 (Pin_33), U2.22 (A15), U3.18 (A16)
- net A17: now also J4.35 (Pin_35), U2.21 (A16), U3.19 (A17)
- net A18: now also J4.37 (Pin_37), U2.20 (A17), U3.20 (A18)
- net A19: now also J4.39 (Pin_39), U2.19 (A18), U3.21 (A19)
- net A2: now also J4.5 (Pin_5), U2.4 (A1), U3.1 (A2), U4.4 (A2)
- net A20: now also J4.41 (Pin_41), U2.18 (A19), U3.22 (A20)
- net A21: now also J4.43 (Pin_43), U3.13 (A21)
- net A3: now also J4.7 (Pin_7), U2.3 (A2), U3.2 (A3), U4.6 (A3)
- net A4: now also J4.9 (Pin_9), U2.2 (A3), U3.3 (A4), U4.7 (A4)
- net A5: now also J4.11 (Pin_11), U2.1 (A4), U3.4 (A5)
- net A6: now also J4.13 (Pin_13), U2.44 (A5), U3.5 (A6)
- net A7: now also J4.15 (Pin_15), U2.43 (A6), U3.6 (A7)
- net A8: now also J4.17 (Pin_17), U2.42 (A7), U3.7 (A8)
- net A9: now also J4.19 (Pin_19), U2.39 (A8), U3.8 (A9)
- net AS: now also J4.47 (Pin_47), U3.31 (AS)
- net BERR: now also J4.49 (Pin_49), RN1.5 (R4), U3.44 (BERR)
- net BG: now also J4.51 (Pin_51), U3.35 (BG)
- net BGACK: now also J4.53 (Pin_53), RN1.7 (R6), U3.36 (BGACK)
- net BR: now also J4.55 (Pin_55), RN1.8 (R7), U3.37 (BR)
- net CLK: now also J4.4 (Pin_4), U3.38 (CLK)
- net CTSA: now also U4.8 (IP0)
- net CTSB: now also U4.5 (IP1)
- net D0: now also J4.61 (Pin_61), U2.9 (DQ0), U3.30 (D0), U4.28 (D0)
- net D1: now also J4.63 (Pin_63), U2.10 (DQ1), U3.29 (D1), U4.18 (D1)
- net D2: now also J4.64 (Pin_64), U2.13 (DQ2), U3.28 (D2), U4.27 (D2)
- net D3: now also J4.62 (Pin_62), U2.14 (DQ3), U3.27 (D3), U4.19 (D3)
- net D4: now also J4.60 (Pin_60), U2.31 (DQ4), U3.26 (D4), U4.26 (D4)
- net D5: now also J4.58 (Pin_58), U2.32 (DQ5), U3.25 (D5), U4.20 (D5)
- net D6: now also J4.56 (Pin_56), U2.35 (DQ6), U3.24 (D6), U4.25 (D6)
- net D7: now also J4.54 (Pin_54), U2.36 (DQ7), U3.23 (D7), U4.21 (D7)
- net DS: now also J4.32 (Pin_32), U3.32 (DS)
- net DTACK: now also J4.57 (Pin_57), U3.34 (DTACK), U4.10 (DTACK)
- net DUAIACK: now also U4.41 (IACK)
- net DUAIRQ: now also U4.24 (INTR)
- net DUASEL: now also U4.39 (CS)
- net E: now also J4.10 (Pin_10), U3.42 (E)
- net FC0: now also J4.20 (Pin_20), U3.50 (FC0)
- net FC1: now also J4.22 (Pin_22), U3.49 (FC1)
- net FC2: now also J4.24 (Pin_24), U3.48 (FC2)
- net HALT: now also IC1.2 (~{RST}), J4.36 (Pin_36), LED3.1 (K), R4.1, U3.40 (HALT), U3.41 (RESET), U4.38 (RESET)
- net IOSEL: now also J4.16 (Pin_16)
- net IPL0: now also RN1.2 (R1), U3.47 (IPL0)
- net IPL1: now also RN1.3 (R2), U3.45 (IPL1)
- net IPL2: now also RN1.4 (R3), U3.46 (IPL2)
- net IRQ2: now also J4.28 (Pin_28)
- net IRQ3: now also J4.14 (Pin_14)
- net IRQ5: now also J4.26 (Pin_26)
- net IRQ6: now also J4.30 (Pin_30)
- net RAMSEL1: now also U2.6 (CE#)
- net RTSA: now also U4.32 (OP0)
- net RTSB: now also U4.14 (OP1)
- net RW: now also J4.59 (Pin_59), U2.17 (WE#), U3.33 (RW), U4.9 (RW)
- net RXDA: now also U4.35 (RXDA)
- net RXDB: now also U4.11 (RXDB)
- net SPICLK: now also U4.30 (OP4)
- net SPICS: now also U4.31 (OP2)
- net SPIMISO: now also U4.40 (IP2)
- net SPIMOSI: now also U4.29 (OP6)
- net TXDA: now also U4.33 (TXDA)
- net TXDB: now also U4.13 (TXDB)
- net VCC: now also J3.5 (Pin_5), JP1.2 (B), JP2.2 (B), U1.32 (VCC), Y1.8 (Vcc), Y2.8 (Vcc), IC1.3 (VCC), J4.2 (Pin_2), J6.1 (Pin_1), R1.1, R5.1, RN1.1 (common), U2.11 (VCC_1), U2.33 (VCC_2), U2.40 (CE2), U3.15 (VCC), U4.44 (VCC)
- net VPA: now also J4.8 (Pin_8), R5.2, RN1.6 (R5), U3.43 (VPA)
- net WR: now also U2.41 (OE#)
- net GPIO0: now reaches U5.35 (I/O)
- net GPIO0: now also J4.38 (Pin_38)
- net GPIO1: now reaches U5.36 (I/O)
- net GPIO1: now also J4.40 (Pin_40)
- net GPIO2: now reaches U5.37 (I/O)
- net GPIO2: now also J4.42 (Pin_42)
- net GPIO3: now reaches U5.39 (I/O)
- net GPIO3: now also J4.44 (Pin_44)
- net GPIO4: now reaches U5.40 (I/O)
- net GPIO4: now also J4.46 (Pin_46)
- net GPIO5: now reaches U5.41 (I/O)
- net GPIO5: now also J4.48 (Pin_48)
- net GPIO6: now reaches U5.52 (I/O)
- net GPIO6: now also J4.50 (Pin_50)
- net GPIO7: now reaches U5.57 (I/O)
- net GPIO7: now also J4.52 (Pin_52)
- net at R2.1: now also U4.16 (OP5)
- net at R3.1: now also U4.15 (OP3)
- net at Y2.5 (OUT): now also U4.36 (X1/CLK)
- net at R2.2: now also LED1.2 (A)
- net at R3.2: now also LED2.2 (A)
- removed net +5V: C1.1, C1.2, C10.1, C10.2, C11.2, C12.1, C12.2, C13.1, C13.2, C14.1, C14.2, C15.1, C15.2, C16.1, C16.2, C17.1, C17.2, C2.1, C2.2, C3.1, C3.2, C4.1, C4.2, C5.1, C5.2, C6.1, C6.2, C7.1, C7.2, C8.1, C8.2, C9.1, C9.2, J1.1 (Pin_1), J2.1 (Pin_1), J3.5 (Pin_5), J3.6 (Pin_6), J5.10 (Pin_10), J5.2 (Pin_2), JP1.2 (B), JP2.2 (B), SW1.1, U1.16 (GND), U1.32 (VCC), U5.19 (GND), U5.32 (GND), U5.42 (GND), U5.47 (GND), U5.59 (GND), U5.7 (GND), U5.72 (GND), U5.82 (GND), Y1.4 (GND), Y1.8 (Vcc), Y2.4 (GND), Y2.8 (Vcc)
- net OE1/I: no longer names the net of U5.84 (OE1/I)
- new net: C1.1, C1.2, C10.1, C10.2, C2.1, C2.2, C3.1, C3.2, C4.1, C4.2, C5.1, C5.2, C6.1, C6.2, C7.1, C7.2, C8.1, C8.2, C9.1, C9.2
- new net: LED3.2 (A), R1.2
- new net: C12.1, C12.2, C13.1, C13.2, C14.1, C14.2, C15.1, C15.2, C16.1, C16.2, C17.1, C17.2
- new net: LED4.2 (A), R4.2
- new net GND: C11.2, IC1.1 (GND), J1.1 (Pin_1), J2.1 (Pin_1), J3.6 (Pin_6), J4.6 (Pin_6), J5.10 (Pin_10), J5.2 (Pin_2), J6.2 (Pin_2), LED1.1 (K), LED2.1 (K), LED4.1 (K), SW1.1, U1.16 (GND), U2.12 (VSS_1), U2.34 (VSS_2), U3.17 (GND), U3.39 (GND), U4.22 (GND), U4.3 (IP3), U4.42 (IP5), U4.43 (IP4), U5.19 (GND), U5.32 (GND), U5.42 (GND), U5.47 (GND), U5.59 (GND), U5.7 (GND), U5.72 (GND), U5.82 (GND), Y1.4 (GND), Y2.4 (GND)
- no-connect marks 39 -> 34
Other:
- moved on the sheet: U5

Commit message: Initial board routing
Parts:
- added C20: 470uF, Capacitor_THT:CP_Radial_D10.0mm_P3.50mm, symbol Device:C_Polarized
- added C21: 100uF, Capacitor_THT:CP_Radial_D5.0mm_P2.50mm, symbol Device:C_Polarized
Connections:
- net GND: now also C1.2, C10.2, C12.2, C13.2, C14.2, C15.2, C16.2, C17.2, C2.2, C3.2, C4.2, C5.2, C6.2, C7.2, C8.2, C9.2, C20.2, C21.2
- net VCC: now also C1.1, C10.1, C12.1, C13.1, C14.1, C15.1, C16.1, C17.1, C2.1, C3.1, C4.1, C5.1, C6.1, C7.1, C8.1, C9.1, C20.1, C21.1
Other:
- moved on the sheet: J6

Commit message: Fabrication
Parts:
- removed H1, H2, H3, H4: MountingHole, MountingHole:MountingHole_3.2mm_M3, symbol Mechanical:MountingHole
- added H1, H2, H3, H4: MountingHole_Pad, MountingHole:MountingHole_3.2mm_M3_Pad_Via, symbol Mechanical:MountingHole_Pad
- added J7: USB_C_Receptacle_PowerOnly_6P, Connector_USB:USB_C_Receptacle_GCT_USB4125-xx-x_6P_TopMnt_Horizontal, symbol Connector:USB_C_Receptacle_PowerOnly_6P
- added R6, R7: 5K1, Resistor_SMD:R_0805_2012Metric_Pad1.20x1.40mm_HandSolder, symbol Device:R
- added U6: TPS22929D, Package_TO_SOT_SMD:SOT-23-6, symbol Power_Management:TPS22929D
- renumbered SW1 to RESET1
Connections:
- net GND: now also H1.1, H2.1, H3.1, H4.1, J7.A12 (GND), J7.B12 (GND), J7.S1 (SHIELD), R6.2, R7.2, U6.2 (GND), U6.5 (GND)
- net VCC: now also U6.1 (VOUT)
- new net: J7.A5 (CC1), R6.1
- new net: J7.A9 (VBUS), J7.B9 (VBUS), U6.3 (ON), U6.4 (VIN), U6.6 (VIN)
- new net: J7.B5 (CC2), R7.1
Other:
- moved on the sheet: C20, C21, J6

Commit message: First pld program
Other:
- note added: "Delete IRQ5 and IRQ6"
- note added: "Need to add A17 (10) and VPA_n (60)"
Changed lines of the file:
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@@
 	(generator_version "9.0")
 	(paper "A3")
+	(text "Need to add A17 (10) and VPA_n (60)"
+		(exclude_from_sim no)
+		(at 290.576 53.594 0)
+		(effects
+			(font
+				(size 1.27 1.27)
+			)
+		)
+	)
+	(text "Delete IRQ5 and IRQ6"
+		(exclude_from_sim no)
+		(at 285.496 56.134 0)
+		(effects
+			(font
+				(size 1.27 1.27)
+			)
+		)
+	)
 	(junction
 		(at 312.42 203.2)
